Commit message: Added Laser Sensor to GAzebo Files, URDF Data and updated project name in launch files

File: urdf/simple_robot_LIDAR.xacro (robot description, xacro)
@@ -1,13 +1,13 @@
 <?xml version="1.0"?>
-<robot name="simple_robot_custom_ctlr" xmlns:xacro="http://www.ros.org/wiki/xacro">
+<robot name="simple_robot_LIDAR" xmlns:xacro="http://www.ros.org/wiki/xacro">
     <!-- if modifications are made to this file, update the simple_robot.urdf file with the following command:
-    rosrun xacro xacro simple_robot_custom_ctlr.xacro > simple_robot_custom_ctlr.urdf
+    rosrun xacro xacro simple_robot_LIDAR.xacro > simple_robot_LIDAR.urdf
     -->
     <xacro:property name="PI" value="3.1415926535897931"/>
     <!-- Import all Gazebo-customization elements, including Gazebo colors -->
-    <xacro:include filename="$(find simple_robot_custom_ctlr)/urdf/simple_robot_custom_ctlr.gazebo" />
+    <xacro:include filename="$(find simple_robot_LIDAR)/urdf/simple_robot_LIDAR.gazebo" />
     <!-- Import Rviz colors -->
-    <xacro:include filename="$(find simple_robot_custom_ctlr)/urdf/materials.xacro" />
-    <xacro:simple_robot_custom_ctlr_gazebo />
+    <xacro:include filename="$(find simple_robot_LIDAR)/urdf/materials.xacro" />
+    <xacro:simple_robot_LIDAR_gazebo />
     <static>false</static>
     <!-- Start of Links - first link must be a non-inertial link -->
@@ -91,5 +91,32 @@
         </visual>
     </link>
+  <!-- Hokuyo Laser -->
+  <link name="hokuyo_link">
+    <collision>
+      <origin xyz="0 0 0" rpy="0 0 0"/>
+      <geometry>
+    <box size="0.1 0.1 0.1"/>
+      </geometry>
+    </collision>
+    <visual>
+      <origin xyz="0 0 0" rpy="0 0 0"/>
+      <geometry>
+        <mesh filename="package://simple_robot_LIDAR/meshes/hokuyo.dae"/>
+      </geometry>
+    </visual>
+    <inertial>
+      <mass value="1e-5" />
+      <origin xyz="0 0 0" rpy="0 0 0"/>
+      <inertia ixx="1e-6" ixy="0" ixz="0" iyy="1e-6" iyz="0" izz="1e-6" />
+    </inertial>
+  </link>
     <!-- Start of Joints - connecting all links together -->
+<joint name="hokuyo_joint" type="fixed">
+    <axis xyz="0 1 0" />
+    <origin xyz="0 0 .5" rpy="0 0 0"/>
+    <parent link="base_link"/>
+    <child link="hokuyo_link"/>
+        <dynamics damping="0.7"/>
+  </joint>
     <joint name="joint0" type="fixed">
         <parent link="base_link"/>

Commit message: Updated Laser Position, included laser scan in RVIZ

File: urdf/simple_robot_LIDAR.xacro (robot description, xacro)
@@ -114,5 +114,5 @@
 <joint name="hokuyo_joint" type="fixed">
     <axis xyz="0 1 0" />
-    <origin xyz="0 0 .5" rpy="0 0 0"/>
+    <origin xyz="-0.1 0 .1" rpy="0 0 ${PI}"/>
     <parent link="base_link"/>
     <child link="hokuyo_link"/>
